File: electronics/carte_bto/adaptateur_3v3_5v.kicad_sch (KiCad schematic)
At the start: 40 parts, among them Q1 MMBT2222A, Q2 MMBT2222A, Q3 MMBT2222A, Q4 MMBT2222A, Q5 MMBT2222A, Q6 MMBT2222A, Q7 MMBT2222A, Q8 MMBT2222A

Commit message: BTO schematic: cleanup and documentation
Connections:
- net DATA_IN1 renamed IN1
- net DATA_IN2 renamed IN2
- net DATA_IN3 renamed IN3
- net DATA_IN4 renamed IN4
- net DATA_IN5 renamed IN5
- net DATA_IN6 renamed IN6
- net DATA_IN7 renamed IN7
- net DATA_IN8 renamed IN0
- net DATA_OUT1 renamed OUT1
- net DATA_OUT2 renamed OUT2
- net DATA_OUT3 renamed OUT3
- net DATA_OUT4 renamed OUT4
- net DATA_OUT5 renamed OUT5
- net DATA_OUT6 renamed OUT6
- net DATA_OUT7 renamed OUT7
- net DATA_OUT8 renamed OUT0
Other:
- note added: "Adaptation de niveau: entrée ≥3.3V, sortie 5V"
- note added: "Ce même modèle est répetté sur chacun des 8 bits du bus. Les montages sont tous les mêmes à l’exception du bit sur lequel il est installé (soit les labels INx et OUTx, où x est l’indice du bit)."
- note added: "Pour le montage transistor: - Si entrée = 0V => transistor passant => sortie = 0V - Si entrée ≥ 3.3V => transistor bloqué => sortie = 5V"
- note added: "Signal numérique (3.3V ou 5V) envoyé par le micro-contrôleur"
- note added: "Une diode pour ne pas tirer de courant sur le micro-contrôleur, et juste garder l’écart de tension à 3.3V."
- moved on the sheet: D1, D2, D3, D4, D5, D6, D7, D8, Q1, Q2, Q3, Q4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

Commit message: BTO: minor schematic fixes & PCB routing.
backup

BTO: Minor fixes on schematic & PCB routing.
Parts:
- R34: renamed from R4; footprint (none) -> Resistor_SMD:R_0805_2012Metric
- R35: renamed from R6; footprint (none) -> Resistor_SMD:R_0805_2012Metric
- R36: renamed from R8; footprint (none) -> Resistor_SMD:R_0805_2012Metric
- R37: renamed from R5; footprint (none) -> Resistor_SMD:R_0805_2012Metric
- R38: renamed from R7; footprint (none) -> Resistor_SMD:R_0805_2012Metric
- R39: renamed from R9; footprint (none) -> Resistor_SMD:R_0805_2012Metric
- R40: renamed from R10; footprint (none) -> Resistor_SMD:R_0805_2012Metric
- R41: renamed from R12; footprint (none) -> Resistor_SMD:R_0805_2012Metric
- R42: renamed from R14; footprint (none) -> Resistor_SMD:R_0805_2012Metric
- R43: renamed from R11; footprint (none) -> Resistor_SMD:R_0805_2012Metric
- R44: renamed from R13; footprint (none) -> Resistor_SMD:R_0805_2012Metric
- R45: renamed from R15; footprint (none) -> Resistor_SMD:R_0805_2012Metric
- R46: renamed from R16; footprint (none) -> Resistor_SMD:R_0805_2012Metric
- R47: renamed from R18; footprint (none) -> Resistor_SMD:R_0805_2012Metric
- R48: renamed from R23; footprint (none) -> Resistor_SMD:R_0805_2012Metric
- R49: renamed from R20; footprint (none) -> Resistor_SMD:R_0805_2012Metric
- R50: renamed from R25; footprint (none) -> Resistor_SMD:R_0805_2012Metric
- R51: renamed from R27; footprint (none) -> Resistor_SMD:R_0805_2012Metric
- R52: renamed from R17; footprint (none) -> Resistor_SMD:R_0805_2012Metric
- R53: renamed from R19; footprint (none) -> Resistor_SMD:R_0805_2012Metric
- R54: renamed from R21; footprint (none) -> Resistor_SMD:R_0805_2012Metric
- R55: renamed from R22; footprint (none) -> Resistor_SMD:R_0805_2012Metric
- R56: renamed from R24; footprint (none) -> Resistor_SMD:R_0805_2012Metric
- R57: renamed from R26; footprint (none) -> Resistor_SMD:R_0805_2012Metric
- renumbered D2 to D10, D3 to D11, D4 to D12, D8 to D13, D5 to D14, D6 to D15, D7 to D16, D1 to D9, Q1 to Q11, Q2 to Q12, Q3 to Q13, Q4 to Q14, Q5 to Q15, Q8 to Q16, Q6 to Q17, Q7 to Q18

Commit message: BTO: more fixes & PCB cleanup
Connections:
- net 3V3 renamed REF
Changed lines of the file:
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@@
 		)
 	)
-	(hierarchical_label "3V3"
+	(hierarchical_label "REF"
 		(shape input)
 		(at 200.66 99.06 180)
@@
 		)
 	)
-	(hierarchical_label "3V3"
+	(hierarchical_label "REF"
 		(shape input)
 		(at 99.06 99.06 180)
@@
 		)
 	)
-	(hierarchical_label "3V3"
+	(hierarchical_label "REF"
 		(shape input)
 		(at 172.72 123.19 180)
@@
 		)
 	)
-	(hierarchical_label "3V3"
+	(hierarchical_label "REF"
 		(shape input)
 		(at 223.52 123.19 180)
@@
 		)
 	)
-	(hierarchical_label "3V3"
+	(hierarchical_label "REF"
 		(shape input)
 		(at 182.88 53.34 180)
@@
 		)
 	)
-	(hierarchical_label "3V3"
+	(hierarchical_label "REF"
 		(shape input)
 		(at 71.12 123.19 180)
@@
 		)
 	)
-	(hierarchical_label "3V3"
+	(hierarchical_label "REF"
 		(shape input)
 		(at 121.92 123.19 180)
@@
 		)
 	)
-	(hierarchical_label "3V3"
+	(hierarchical_label "REF"
 		(shape input)
 		(at 149.86 99.06 180)

Commit message: BTO: Changed footprints to handsoldering verions, redid PCB routing
Parts:
- removed D10, D11, D12, D13, D14, D15, D16, D9: 1N4148WT, Diode_SMD:D_SOD-523, symbol Diode:1N4148WT
- removed Q11, Q12, Q13, Q14, Q15, Q16, Q17, Q18: MMBT2222A, Package_TO_SOT_SMD:SOT-23, symbol Transistor_BJT:MMBT2222A
- removed R34, R36, R37, R39, R40, R42, R43, R45, R46, R48, R49, R51, R52, R54, R55, R57: 10k, Resistor_SMD:R_0805_2012Metric, symbol Device:R
- removed R35, R38, R41, R44, R47, R50, R53, R56: 22k, Resistor_SMD:R_0805_2012Metric, symbol Device:R
Other:
- note removed: "Adaptation de niveau: entrée ≥3.3V, sortie 5V"
- note removed: "Ce même modèle est répetté sur chacun des 8 bits du bus. Les montages sont tous les mêmes à l’exception du bit sur lequel il est installé (soit les labels INx et OUTx, où x est l’indice du bit)."
- note removed: "Pour le montage transistor: - Si entrée = 0V => transistor passant => sortie = 0V - Si entrée ≥ 3.3V => transistor bloqué => sortie = 5V"
- note removed: "Signal numérique (3.3V ou 5V) envoyé par le micro-contrôleur"
- note removed: "Une diode pour ne pas tirer de courant sur le micro-contrôleur, et juste garder l’écart de tension à 3.3V."
