File: electronics/carte_bto/carte_bto.kicad_sch (KiCad schematic)
At the start: 70 parts, among them J1 DIN41612_02x32_AB, J2 Conn_01x01, J3 Conn_01x01, J4 Conn_01x01, J5 Conn_01x01, J6 Conn_01x01, Q1 MMBT2222A, Q2 MMBT2222A, U1 74AHC541, U2 LTC1859IG_PBF, U3 LT6654AIS6-2.5_TRPBF, U4 74AHC541, U5 L78L05_SOT89

Commit message: BTO: added 0Ω resistors for a net class hack.
Parts:
- added R82, R83: 0, Resistor_SMD:R_0805_2012Metric, symbol Device:R_Small
- Z9: footprint Diode_SMD:D_SOD-882 -> Diode_SMD:D_SOD-523
Connections:
- net +5V: now also R82.2, R83.2; no longer U1.20 (VCC), U4.20 (VCC)
- new net: R82.1, U4.20 (VCC)
- new net: R83.1, U1.20 (VCC)
Changed lines of the file:
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@@
 	(text "Buffer 8 bits:\n- protection surtensions\n- sortie haute impédence\n   quand hors-tension."
 		(exclude_from_sim no)
-		(at 176.53 22.86 0)
+		(at 173.99 22.86 0)
 		(effects
 			(font
@@
 			)
 		)
-		(property "Footprint" "Diode_SMD:D_SOD-882"
+		(property "Footprint" "Diode_SMD:D_SOD-523"
 			(at 64.77 181.61 0)
 			(effects
@@
 	)
 	(symbol
+		(lib_id "power:+5V")
+		(at 77.47 22.86 0)
+		(unit 1)
+		(exclude_from_sim no)
+		(in_bom yes)
+		(on_board yes)
+		(dnp no)
+		(property "Reference" "#PWR012"
+			(at 77.47 26.67 0)
+			(effects
+				(font
+					(size 1.27 1.27)
+				)
+				(hide yes)
+			)
+		)
+		(property "Value" "+5V"
+			(at 77.47 19.05 0)
+			(effects
+				(font
+					(size 1.27 1.27)
+				)
+			)
+		)
+		(property "Footprint" ""
+			(at 77.47 22.86 0)
+			(effects
+				(font
+					(size 1.27 1.27)
+				)
+				(hide yes)
+			)
+		)
+		(property "Datasheet" ""
+			(at 77.47 22.86 0)
+			(effects
+				(font
+					(size 1.27 1.27)
+				)
+				(hide yes)
+			)
+		)
+		(property "Description" "Power symbol creates a global label with name \"+5V\""
+			(at 77.47 22.86 0)
+			(effects
+				(font
+					(size 1.27 1.27)
+				)
+				(hide yes)
+			)
+		)
+		(pin "1"
+		)
+		(instances
+			(project "carte_bto"
+				(path "/b37cf66c-5553-4962-b28a-30df843edffa"
+					(reference "#PWR012")
+					(unit 1)
+				)
+			)
+		)
+	)
+	(symbol
 		(lib_id "power:PWR_FLAG")
 		(at 227.33 125.73 0)
@@
 	)
 	(symbol
-		(lib_id "power:+5V")
-		(at 72.39 22.86 0)
-		(unit 1)
-		(exclude_from_sim no)
-		(in_bom yes)
-		(on_board yes)
-		(dnp no)
-		(property "Reference" "#PWR030"
-			(at 72.39 26.67 0)
-			(effects
-				(font
-					(size 1.27 1.27)
-				)
-				(hide yes)
-			)
-		)
-		(property "Value" "+5V"
-			(at 72.39 19.05 0)
-			(effects
-				(font
-					(size 1.27 1.27)
-				)
-			)
-		)
-		(property "Footprint" ""
-			(at 72.39 22.86 0)
-			(effects
-				(font
-					(size 1.27 1.27)
-				)
-				(hide yes)
-			)
-		)
-		(property "Datasheet" ""
-			(at 72.39 22.86 0)
-			(effects
-				(font
-					(size 1.27 1.27)
-				)
-				(hide yes)
-			)
-		)
-		(property "Description" "Power symbol creates a global label with name \"+5V\""
-			(at 72.39 22.86 0)
-			(effects
-				(font
-					(size 1.27 1.27)
-				)
-				(hide yes)
-			)
-		)
-		(pin "1"
-		)
-		(instances
-			(project "carte_bto"
-				(path "/b37cf66c-5553-4962-b28a-30df843edffa"
-					(reference "#PWR030")
-					(unit 1)
-				)
-			)
-		)
-	)
-	(symbol
 		(lib_id "Connector:DIN41612_02x32_AB")
 		(at 50.8 128.27 0)
@@
 	)
 	(symbol
+		(lib_id "Device:R_Small")
+		(at 207.01 22.86 90)
+		(unit 1)
+		(exclude_from_sim no)
+		(in_bom yes)
+		(on_board yes)
+		(dnp no)
+		(property "Reference" "R82"
+			(at 207.01 21.082 90)
+			(effects
+				(font
+					(size 1.016 1.016)
+				)
+			)
+		)
+		(property "Value" "0"
+			(at 207.01 22.86 90)
+			(effects
+				(font
+					(size 1.27 1.27)
+				)
+			)
+		)
+		(property "Footprint" "Resistor_SMD:R_0805_2012Metric"
+			(at 207.01 22.86 0)
+			(effects
+				(font
+					(size 1.27 1.27)
+				)
+				(hide yes)
+			)
+		)
+		(property "Datasheet" "~"
+			(at 207.01 22.86 0)
+			(effects
+				(font
+					(size 1.27 1.27)
+				)
+				(hide yes)
+			)
+		)
+		(property "Description" "Resistor, small symbol"
+			(at 207.01 22.86 0)
+			(effects
+				(font
+					(size 1.27 1.27)
+				)
+				(hide yes)
+			)
+		)
+		(pin "1"
+		)
+		(pin "2"
+		)
+		(instances
+			(project ""
+				(path "/b37cf66c-5553-4962-b28a-30df843edffa"
+					(reference "R82")
+					(unit 1)
+				)
+			)
+		)
+	)
+	(symbol
 		(lib_id "power:GNDD")
 		(at 217.17 69.85 0)
@@
 	)
 	(symbol
+		(lib_id "Device:R_Small")
+		(at 74.93 22.86 90)
+		(unit 1)
+		(exclude_from_sim no)
+		(in_bom yes)
+		(on_board yes)
+		(dnp no)
+		(property "Reference" "R83"
+			(at 74.93 21.082 90)
+			(effects
+				(font
+					(size 1.016 1.016)
+				)
+			)
+		)
+		(property "Value" "0"
+			(at 74.93 22.86 90)
+			(effects
+				(font
+					(size 1.27 1.27)
+				)
+			)
+		)
+		(property "Footprint" "Resistor_SMD:R_0805_2012Metric"
+			(at 74.93 22.86 0)
+			(effects
+				(font
+					(size 1.27 1.27)
+				)
+				(hide yes)
+			)
+		)
+		(property "Datasheet" "~"
+			(at 74.93 22.86 0)
+			(effects
+				(font
+					(size 1.27 1.27)
+				)
+				(hide yes)
+			)
+		)
+		(property "Description" "Resistor, small symbol"
+			(at 74.93 22.86 0)
+			(effects
+				(font
+					(size 1.27 1.27)
+				)
+				(hide yes)
+			)
+		)
+		(pin "1"
+		)
+		(pin "2"
+		)
+		(instances
+			(project "carte_bto"
+				(path "/b37cf66c-5553-4962-b28a-30df843edffa"
+					(reference "R83")
+					(unit 1)
+				)
+			)
+		)
+	)
+	(symbol
 		(lib_id "power:GND1")
 		(at 125.73 157.48 0)
@@
 		(dnp no)
 		(property "Reference" "U1"
-			(at 72.39 24.13 0)
+			(at 72.39 24.892 0)
 			(effects
 				(font
@@
 	(symbol
 		(lib_id "power:+5V")
-		(at 204.47 22.86 0)
+		(at 209.55 22.86 0)
 		(unit 1)
 		(exclude_from_sim no)
@@
 		(dnp no)
 		(property "Reference" "#PWR031"
-			(at 204.47 26.67 0)
+			(at 209.55 26.67 0)
 			(effects
 				(font
@@
 		)
 		(property "Value" "+5V"
-			(at 204.47 19.05 0)
+			(at 209.55 19.05 0)
 			(effects
 				(font
@@
 		)
 		(property "Footprint" ""
-			(at 204.47 22.86 0)
+			(at 209.55 22.86 0)
 			(effects
 				(font
@@
 		)
 		(property "Datasheet" ""
-			(at 204.47 22.86 0)
+			(at 209.55 22.86 0)
 			(effects
 				(font
@@
 		)
 		(property "Description" "Power symbol creates a global label with name \"+5V\""
-			(at 204.47 22.86 0)
+			(at 209.55 22.86 0)
 			(effects
 				(font
@@
 		(dnp no)
 		(property "Reference" "U4"
-			(at 204.47 24.13 0)
+			(at 204.47 24.892 0)
 			(effects
 				(font

Commit message: BTO: Changed footprints to handsoldering verions, redid PCB routing
Parts:
- removed C1, C2, C3, C4: 4.7µF, Capacitor_SMD:C_0805_2012Metric, symbol Device:C_Small
- removed C10, C11, C26, C7, C8, C9: 100nF, Capacitor_SMD:C_0805_2012Metric, symbol Device:C_Small
- removed C6: 10µF, Capacitor_SMD:C_0805_2012Metric, symbol Device:C_Small
- removed CT1, CT2, CT3, CT4: 10µF, Capacitor_Tantalum_SMD:CP_EIA-2012-12_Kemet-R, symbol Device:C_Polarized_Small
- removed D24, D25: SMAJ15A, Diode_SMD:D_SOD-323_HandSoldering, symbol Diode:SMAJ15A
- removed D27: SMAJ12A, Diode_SMD:D_SOD-323_HandSoldering, symbol Diode:SMAJ12A
- removed J1: DIN41612_02x32_AB, Connector_DIN:DIN41612_B_2x32_Male_Horizontal_THT, symbol Connector:DIN41612_02x32_AB
- removed J2, J3, J4, J5, J6: Conn_01x01, imported_components:HIRSCHMANN_930224100, symbol 930224100:930224100
- removed LD1, LD2, LD3, LD5: LED_Small, LED_SMD:LED_0805_2012Metric, symbol Device:LED_Small
- removed LD4, LD6: LED, LED_SMD:LED_0805_2012Metric, symbol Device:LED
- removed Q1, Q2: MMBT2222A, Package_TO_SOT_SMD:SOT-23, symbol Transistor_BJT:MMBT2222A
- removed R1: 3.3k, Resistor_SMD:R_0805_2012Metric, symbol Device:R_Small
- removed R2, R3, R4: 5.1k, Resistor_SMD:R_0805_2012Metric, symbol Device:R_Small
- removed R5, R8: 3.3k, Resistor_SMD:R_0805_2012Metric, symbol Device:R
- removed R6, R9: 22k, Resistor_SMD:R_0805_2012Metric, symbol Device:R
- removed R82, R83: 0, Resistor_SMD:R_0805_2012Metric, symbol Device:R_Small
- removed U1, U4: 74AHC541, Package_SO:TSSOP-20_4.4x5mm_P0.4mm, symbol 74xx:74AHC541
- removed U2: LTC1859IG_PBF, imported_components:SSOP-28_G, symbol LTC1859IG_PBF:LTC1859IG_PBF
- removed U3: LT6654AIS6-2.5_TRPBF, imported_components:SOT95P280X100-6N, symbol LT6654AIS6-2.5_TRPBF:LT6654AIS6-2.5_TRPBF
- removed U5: L78L05_SOT89, Package_TO_SOT_SMD:SOT-89-3, symbol Regulator_Linear:L78L05_SOT89
- removed Z1, Z13, Z14, Z15, Z16, Z17, Z18, Z19, Z2, Z20, Z3, Z4, Z5, Z6, Z7, Z8: PESD5V0L1UL, Diode_SMD:D_SOD-882, symbol Diode:PESD5V0L1UL
- removed Z9: PESD5V0L1UL, Diode_SMD:D_SOD-523, symbol Diode:PESD5V0L1UL
- C1: renamed from C20; footprint Capacitor_SMD:C_0805_2012Metric -> Capacitor_SMD:C_0805_2012Metric_Pad1.18x1.45mm_HandSolder
- C2: renamed from C21; footprint Capacitor_SMD:C_0805_2012Metric -> Capacitor_SMD:C_0805_2012Metric_Pad1.18x1.45mm_HandSolder
- C3: renamed from C22; footprint Capacitor_SMD:C_0805_2012Metric -> Capacitor_SMD:C_0805_2012Metric_Pad1.18x1.45mm_HandSolder
- C4: renamed from C23; footprint Capacitor_SMD:C_0805_2012Metric -> Capacitor_SMD:C_0805_2012Metric_Pad1.18x1.45mm_HandSolder
- C5: renamed from C24; footprint Capacitor_SMD:C_0805_2012Metric -> Capacitor_SMD:C_0805_2012Metric_Pad1.18x1.45mm_HandSolder
- C6: renamed from C25; footprint Capacitor_SMD:C_0805_2012Metric -> Capacitor_SMD:C_0805_2012Metric_Pad1.18x1.45mm_HandSolder
- R1: renamed from R7; footprint Resistor_SMD:R_0805_2012Metric -> Resistor_SMD:R_0805_2012Metric_Pad1.20x1.40mm_HandSolder
Connections:
- net SPI.cipo renamed ADC 16 bits 8 voies/SPI_CIPO
- net SPI.copi renamed ADC 16 bits 8 voies/SPI_COPI
- net SPI.cs renamed ADC 16 bits 8 voies/SPI_CS
- net SPI.sck renamed ADC 16 bits 8 voies/SPI_SCK
- net adc_busy renamed ADC 16 bits 8 voies/~{BUSY}
- no-connect marks 11 -> 3
Other:
- removed sheet Adaptateur 3v3 - 5v 8voies (1)
- removed sheet Adaptateur 3v3 - 5v 8voies (2)
- removed sheet Protections 8voies analogiques
- added sheet ADC 16 bits 8 voies (adc_16_bits_8_voies.kicad_sch)
- added sheet Bus donnée (bus_donnee.kicad_sch)
- added sheet Bus d’adresse (bus_adresse.kicad_sch)
- added sheet Bus fond de panier (bus_fond_de_panier.kicad_sch)
- note removed: "ADC 16 bits, 8 voies SPI"
- note removed: "Activer les sorties quand la carte est sous tension (+ LED de status)."
- note removed: "Activer les sorties quand la carte est sous tension. (+ LED de status)"
- note removed: "Buffer 8 bits: - protection surtensions - Sortie haute impédence quand hors-tension."
- note removed: "Buffer 8 bits: - protection surtensions - sortie haute impédence quand hors-tension."
- note removed: "Bus fond de panier"
- note removed: "Connexion vers bus fond de panier"
- note removed: "Conversion analogique -> numérique"
- note removed: "On relie le ground de l’ADC sur un autre plan de masse que le reste de la carte, afin de réduire les bruits parasites."
- note removed: "Protection décharges électro-statiques"
- note removed: "Tension de référence stable (2.5V)"
- moved on the sheet: A1, C1, C2, C3, C4, C5, C6, R1
